File: Double-DigiPot-with-IR/Double-DigiPot-with-IR.kicad_pcb (KiCad board)
At the start: 2 copper layers, 19 parts, among them J1 Conn_01x09_Pin, SW1 SW_Push_DPDT, SW2 EVQ-P7A01P, SW3 EVQ-P7A01P, U1 ATtiny404-SS, U2 MCP4561T-503E/MS, U3 MCP4561T-503E/MS, U4 TSOP382xx

Commit message: Updated PCB
Parts:
- added C5: 47u, Capacitor_SMD:C_1210_3225Metric, F.Cu at (203.6, 88.2)
- added C6: 47u, Capacitor_SMD:C_1210_3225Metric, F.Cu at (198.2, 88.2)
- added TP1: TestPoint, TestPoint:TestPoint_Pad_D4.0mm, F.Cu at (202.6, 107.8)
- added TP2: TestPoint, TestPoint:TestPoint_Pad_D4.0mm, F.Cu at (202.6, 102.2)
- added U5: AMS1117-3.3, Package_TO_SOT_SMD:SOT-223-3_TabPin2, F.Cu at (202.0, 94.8)
- J1: footprint Connector_Molex:Molex_Pico-Clasp_202396-0907_1x09-1MP_P1.00mm_Horizontal -> Connector_PinSocket_2.54mm:PinSocket_1x09_P2.54mm_Vertical
- U2, U3: value MCP4561T-503E/MS -> MCP4561T-103E/MS
- moved R2 50.7 mm to (184.2, 102.6), turned to 180 degrees
- moved J1 50.7 mm to (202.2, 77.5), turned to -90 degrees
- moved SW3 46.5 mm to (174.6, 95.8), turned to 90 degrees
- moved R1 42.6 mm to (184.2, 105.0), turned to 0 degrees
- moved C2 42.5 mm to (187.5, 88.5)
- moved C3 41.6 mm to (179.0, 88.5)
- moved R5 41.5 mm to (198.5, 103.2), turned to 90 degrees
- moved U1 41.1 mm to (192.0, 103.0)
- moved U2 41.1 mm to (182.5, 90.0)
- moved U3 41.1 mm to (191.0, 90.0)
- moved U4 41.1 mm to (189.5, 129.5)
- moved C4 40.9 mm to (193.5, 126.5)
- moved SW1 40.9 mm to (202.9, 112.8)
- moved D1 40.0 mm to (177.8, 116.8)
- moved SW2 39.4 mm to (174.6, 103.2), turned to 90 degrees
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Connections:
- C1 pad 1: +5V -> 3.3
- C2 pad 2: +5V -> 3.3
- C3 pad 2: +5V -> 3.3
- C4 pad 1: +5V -> 3.3
- R1 pad 1: Net-(U1-PA7) -> Net-(D1-BA)
- R1 pad 2: Net-(D1-BA) -> Net-(U1-PA7)
- R3 pad 2: +5V -> 3.3
- R4 pad 1: +5V -> 3.3
- R6 pad 1: Net-(R6-Pad1) -> Net-(U1-PA1)
- SW1 pad 5: Net-(R6-Pad1) -> Net-(U1-PA1)
- SW1 pad 6: LED pwr -> 3.3
- SW2 pad 1: +5V -> 3.3
- SW2 pad 1*: unconnected-(SW2-Pad1*) -> 3.3
- SW2 pad 2: unconnected-(SW2-Pad2) -> Net-(U1-PA5)
- SW3 pad 1: +5V -> 3.3
- SW3 pad 1*: unconnected-(SW3-Pad1*) -> 3.3
- SW3 pad 2: unconnected-(SW3-Pad2) -> Net-(U1-PA4)
- U1 pad 1: +5V -> 3.3
- U1 pad 11: unconnected-(U1-PA1-Pad11) -> Net-(U1-PA1)
- U1 pad 6: unconnected-(U1-PB3-Pad6) -> Net-(U1-PB3)
- U1 pad 7: Net-(U1-PB2) -> TXD
- U2 pad 1: +5V -> 3.3
- U2 pad 8: +5V -> 3.3
- U3 pad 8: +5V -> 3.3
- U4 pad 1: Net-(U1-PB2) -> Net-(U1-PB3)
- U4 pad 3: +5V -> 3.3
Routing:
- net +5V: track 102.6 -> 0.00 mm, vias 6 -> 0
- net Net-(U1-PA1): track 0.00 -> 45.6 mm, vias 0 -> 2
- net Net-(U1-PB3): track 0.00 -> 29.6 mm
- net Net-(U1-PB1): track 57.3 -> 28.4 mm
- net LED pwr: track 44.8 -> 16.4 mm, vias 0 -> 1
- net Net-(R6-Pad1): track 26.5 -> 0.00 mm
- net Net-(U1-PB2): track 24.3 -> 0.00 mm, vias 2 -> 0
- net Net-(U1-PB0): track 49.1 -> 28.9 mm, vias 2 -> 0
- net 3.3: track 0.00 -> 19.1 mm, vias 0 -> 4
- net TXD: track 0.00 -> 13.5 mm
- net Net-(D1-RA): track 3.60 -> 16.5 mm
- net Rout: track 8.48 -> 19.1 mm
- net GND: track 14.4 -> 24.9 mm, vias 9 -> 11
- net Net-(U1-PA6): track 14.7 -> 4.54 mm
- net /pgm: track 14.3 -> 4.14 mm, vias 3 -> 0
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- added copper zone on F.Cu, net 3.3
Other:
- board outline added: 37.6 x 58.2 mm
