File: Double-DigiPot-with-IR/Double-DigiPot-with-IR.kicad_pcb (KiCad board)
At the start: 2 copper layers, 37.6 x 58.2 mm, 33 parts, among them J1 Conn_01x09_Pin, SW1 SW_Push_DPDT, U1 ATtiny404-SS, U2 MCP4561T-103E/MS, U3 MCP4561T-103E/MS, U4 TSOP382xx, U6 MC78L05_SOT89

Commit message: Digipot V2!!!!
Parts:
- C10, C7, C8, C9: value 100n -> 10u
- R11: renamed from R13; value 4.7k -> 10k
- R12: value 4.7k -> 10k
- renumbered C3 to C2, C2 to C3, R11 to R10, R6 to R2, R2 to R3, R3 to R4, R4 to R5, R5 to R6, R9 to R7, R10 to R9
Routing:
- net GND: track 40.1 -> 42.5 mm, vias 53 -> 55
- net Net-(U1-PB1): track 34.8 -> 33.7 mm
- net TXD: track 24.5 -> 23.5 mm, vias 0 -> 2
- net Net-(U1-PB0): track 35.2 -> 35.7 mm
- net Net-(U1-PA7): track 13.4 -> 13.6 mm, vias 0 -> 1
Other:
- board text added: "GND Lout Rout GND Lin Rin STout STin Vled"
- board text added: "PA0 -> pgm PA1 -> NC PA2 -> NC PA3 -> BLU PA4 -> GRN PA5 -> RED PA6 -> NC PA7 -> SW PB0 -> SCL PB1 -> SDA PB2 -> TXD PB3 -> IR"
- board text added: "R1,2,3 -> 330 R4,5,6 -> 4.7k R7-12 -> 10k C1,2,3,4 -> 100n C5-10 -> 10u"
