File: Double-DigiPot-with-IR/Double-DigiPot-with-IR.kicad_sch (KiCad schematic)
At the start: 19 parts, among them J1 Conn_01x09_Pin, SW1 SW_Push_DPDT, SW2 EVQ-P7A01P, SW3 EVQ-P7A01P, U1 ATtiny404-SS, U2 MCP4561T-503E/MS, U3 MCP4561T-503E/MS, U4 TSOP382xx

Commit message: Updated PCB
Parts:
- added C5, C6: 47u, Capacitor_SMD:C_1210_3225Metric, symbol Device:C_Small
- added TP1, TP2: TestPoint, TestPoint:TestPoint_Pad_D4.0mm, symbol Connector:TestPoint
- added U5: AMS1117-3.3, Package_TO_SOT_SMD:SOT-223-3_TabPin2, symbol Regulator_Linear:AMS1117-3.3
- J1: footprint Connector_Molex:Molex_Pico-Clasp_202396-0907_1x09-1MP_P1.00mm_Horizontal -> Connector_PinSocket_2.54mm:PinSocket_1x09_P2.54mm_Vertical
- U2, U3: value MCP4561T-503E/MS -> MCP4561T-103E/MS
Connections:
- net +5V is gone; now on net 3.3: C1.1, C2.2, C3.2, C4.1, R3.2, R4.1, SW2.1, SW3.1, U1.1 (VCC), U2.1 (HVC/A0), U2.8 (VDD), U3.8 (VDD), U4.3 (Vs)
- net GND: now also C5.2, C6.2, U5.1 (GND)
- net LED pwr: now also C6.1, U5.3 (VI); no longer SW1.6 (C)
- net pgm: now also TP2.1
- net 3.3: now reaches SW2.1*
- net 3.3: now also SW1.6 (C), SW3.1*, C5.1, U5.2 (VO)
- net at SW2.2: now also SW2.2*, U1.3 (PA5)
- net at U1.11 (PA1): now also R6.1, SW1.5 (B)
- net at SW3.2*, U1.2 (PA4): now also SW3.2
- net at U1.6 (PB3): now also U4.1 (OUT)
- net TXD: now reaches U1.7 (PB2)
- net TXD: now also TP1.1; no longer U4.1 (OUT)
