File: Double-DigiPot-with-IR/Double-DigiPot-with-IR.kicad_sch (KiCad schematic)
At the start: 24 parts, among them J1 Conn_01x09_Pin, SW1 SW_Push_DPDT, SW2 EVQ-P7A01P, SW3 EVQ-P7A01P, U1 ATtiny404-SS, U2 MCP4561T-103E/MS, U3 MCP4561T-103E/MS, U4 TSOP382xx, U5 AMS1117-3.3

Commit message: MEGA UPDATE (Redesign) (It might work now)
Parts:
- removed SW2, SW3: EVQ-P7A01P, EVQ_P7_PAN, symbol EdgeSwitch:EVQ-P7A01P
- removed U5: AMS1117-3.3, Package_TO_SOT_SMD:SOT-223-3_TabPin2, symbol Regulator_Linear:AMS1117-3.3
- added C10, C7, C8, C9: 100n, Capacitor_SMD:C_0805_2012Metric_Pad1.18x1.45mm_HandSolder, symbol Device:C
- added R10, R11, R8, R9: 10k, Resistor_SMD:R_0805_2012Metric_Pad1.20x1.40mm_HandSolder, symbol Device:R
- added R12, R13: 4.7k, Resistor_SMD:R_0805_2012Metric_Pad1.20x1.40mm_HandSolder, symbol Device:R
- added TP3: GNDPoint, TestPoint:TestPoint_Pad_D4.0mm, symbol Connector:TestPoint
- added U6: MC78L05_SOT89, Package_TO_SOT_SMD:SOT-89-3_Handsoldering, symbol Regulator_Linear:MC78L05_SOT89
- C1, C2, C3, C4: footprint Capacitor_SMD:C_0805_2012Metric -> Capacitor_SMD:C_0805_2012Metric_Pad1.18x1.45mm_HandSolder
- C5, C6: value 47u -> 10u; footprint Capacitor_SMD:C_1210_3225Metric -> Capacitor_SMD:C_0805_2012Metric_Pad1.18x1.45mm_HandSolder
- R1, R6: value 4.7k -> 330; footprint Resistor_SMD:R_0805_2012Metric -> Resistor_SMD:R_0805_2012Metric_Pad1.20x1.40mm_HandSolder
- R2: value 4.7k -> 330; footprint Capacitor_SMD:C_0805_2012Metric -> Resistor_SMD:R_0805_2012Metric_Pad1.20x1.40mm_HandSolder
- R3, R5: footprint Resistor_SMD:R_0805_2012Metric -> Resistor_SMD:R_0805_2012Metric_Pad1.20x1.40mm_HandSolder
- R4: footprint Capacitor_SMD:C_0805_2012Metric -> Resistor_SMD:R_0805_2012Metric_Pad1.20x1.40mm_HandSolder
- SW1: footprint DigiPot:CONN_S2273_APM -> digiPot:CONN_S2273_APM
- U2, U3: footprint DigiPot:MSOP8_MC_MCH -> digiPot:MSOP8_MC_MCH
Connections:
- net GND: now also R11.1, R12.1, R8.1, TP3.1, U6.2 (GND); no longer U2.7 (P0B), U3.7 (P0B)
- net LED pwr: now also U6.3 (IN)
- net Lin: now also C7.1, R8.2, R9.1; no longer J1.5 (Pin_5)
- net Lout: now also C9.1; no longer J1.8 (Pin_8)
- net Rin: now also C8.1, R10.1, R11.2; no longer J1.4 (Pin_4)
- net Rout: now also C10.1; no longer J1.7 (Pin_7)
- net at U1.3 (PA5): now also R2.1
- net at U1.13 (PA3): now also R1.2
- net at U1.2 (PA4): now also R6.1
- net at U1.4 (PA6): no longer R2.1
- net at U1.5 (PA7): now also SW1.5 (B); no longer R1.2
- net 3.3 renamed 5
- net 5: now also R10.2, R13.1, R9.2, U6.1 (OUT)
- new net: C10.2, J1.7 (Pin_7)
- new net: C8.2, J1.4 (Pin_4)
- new net: C7.2, J1.5 (Pin_5)
- new net: C9.2, J1.8 (Pin_8)
- new net ref: R12.2, R13.2, U2.7 (P0B), U3.7 (P0B)
- now unconnected: U1.11 (PA1)
- no-connect marks 0 -> 3
Other:
- moved on the sheet: J1, R6

Commit message: Digipot V2!!!!
Parts:
- C10, C7, C8, C9: value 100n -> 10u
- R11: renamed from R13; value 4.7k -> 10k
- R12: value 4.7k -> 10k
- renumbered C3 to C2, C2 to C3, R11 to R10, R6 to R2, R2 to R3, R3 to R4, R4 to R5, R5 to R6, R9 to R7, R10 to R9
Changed lines of the file:
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@@
 			)
 		)
-		(property "Value" "100n"
+		(property "Value" "10u"
 			(at 214.63 68.58 90)
 			(show_name no)
@@
 		(dnp no)
 		(fields_autoplaced yes)
-		(property "Reference" "R13"
+		(property "Reference" "R11"
 			(at 246.38 100.33 90)
 			(show_name no)
@@
 			)
 		)
-		(property "Value" "4.7k"
+		(property "Value" "10k"
 			(at 246.38 102.87 90)
 			(show_name no)
@@
 			(project "Double-DigiPot-with-IR"
 				(path "/8790fbe4-afd7-47db-a1db-a7a2fdad799c"
-					(reference "R13")
+					(reference "R11")
 					(unit 1)
 				)
@@
 		(dnp no)
 		(fields_autoplaced yes)
-		(property "Reference" "C3"
+		(property "Reference" "C2"
 			(at 147.32 78.74 90)
 			(show_name no)
@@
 			(project "Double-DigiPot-with-IR"
 				(path "/8790fbe4-afd7-47db-a1db-a7a2fdad799c"
-					(reference "C3")
+					(reference "C2")
 					(unit 1)
 				)
@@
 		(dnp no)
 		(fields_autoplaced yes)
-		(property "Reference" "C2"
+		(property "Reference" "C3"
 			(at 146.05 119.38 90)
 			(show_name no)
@@
 			(project "Double-DigiPot-with-IR"
 				(path "/8790fbe4-afd7-47db-a1db-a7a2fdad799c"
-					(reference "C2")
+					(reference "C3")
 					(unit 1)
 				)
@@
 			)
 		)
-		(property "Value" "100n"
+		(property "Value" "10u"
 			(at 214.63 78.74 90)
 			(show_name no)
@@
 			)
 		)
-		(property "Value" "4.7k"
+		(property "Value" "10k"
 			(at 245.11 111.7599 0)
 			(show_name no)
@@
 			)
 		)
-		(property "Value" "100n"
+		(property "Value" "10u"
 			(at 214.63 73.66 90)
 			(show_name no)
@@
 		(dnp no)
 		(fields_autoplaced yes)
-		(property "Reference" "R5"
+		(property "Reference" "R6"
 			(at 90.17 80.0099 0)
 			(show_name no)
@@
 			(project "Double-DigiPot-with-IR"
 				(path "/8790fbe4-afd7-47db-a1db-a7a2fdad799c"
-					(reference "R5")
+					(reference "R6")
 					(unit 1)
 				)
@@
 		(dnp no)
 		(fields_autoplaced yes)
-		(property "Reference" "R4"
+		(property "Reference" "R5"
 			(at 115.57 52.0699 0)
 			(show_name no)
@@
 			(project "Double-DigiPot-with-IR"
 				(path "/8790fbe4-afd7-47db-a1db-a7a2fdad799c"
-					(reference "R4")
+					(reference "R5")
 					(unit 1)
 				)
@@
 		(dnp no)
 		(fields_autoplaced yes)
-		(property "Reference" "R2"
+		(property "Reference" "R3"
 			(at 101.6 149.86 90)
 			(show_name no)
@@
 			(project "Double-DigiPot-with-IR"
 				(path "/8790fbe4-afd7-47db-a1db-a7a2fdad799c"
-					(reference "R2")
+					(reference "R3")
 					(unit 1)
 				)
@@
 		(dnp no)
 		(fields_autoplaced yes)
-		(property "Reference" "R9"
+		(property "Reference" "R7"
 			(at 199.39 73.6599 0)
 			(show_name no)
@@
 			(project "Double-DigiPot-with-IR"
 				(path "/8790fbe4-afd7-47db-a1db-a7a2fdad799c"
-					(reference "R9")
+					(reference "R7")
 					(unit 1)
 				)
@@
 		(dnp no)
 		(fields_autoplaced yes)
-		(property "Reference" "R10"
+		(property "Reference" "R9"
 			(at 203.2 77.4699 0)
 			(show_name no)
@@
 			(project "Double-DigiPot-with-IR"
 				(path "/8790fbe4-afd7-47db-a1db-a7a2fdad799c"
-					(reference "R10")
+					(reference "R9")
 					(unit 1)
 				)
@@
 		(dnp no)
 		(fields_autoplaced yes)
-		(property "Reference" "R11"
+		(property "Reference" "R10"
 			(at 203.2 86.3599 0)
 			(show_name no)
@@
 			(project "Double-DigiPot-with-IR"
 				(path "/8790fbe4-afd7-47db-a1db-a7a2fdad799c"
-					(reference "R11")
+					(reference "R10")
 					(unit 1)
 				)
@@
 		(in_pos_files yes)
 		(dnp no)
-		(fields_autoplaced yes)
-		(property "Reference" "R3"
-			(at 102.87 53.34 90)
+		(property "Reference" "R4"
+			(at 105.41 52.07 0)
 			(show_name no)
 			(do_not_autoplace no)
@@
 					(size 1.27 1.27)
 				)
+				(justify right)
 			)
 		)
 		(property "Value" "4.7k"
-			(at 105.41 53.34 90)
+			(at 103.886 54.356 0)
 			(show_name no)
 			(do_not_autoplace no)
@@
 					(size 1.27 1.27)
 				)
+				(justify right)
 			)
 		)
@@
 			(project "Double-DigiPot-with-IR"
 				(path "/8790fbe4-afd7-47db-a1db-a7a2fdad799c"
-					(reference "R3")
+					(reference "R4")
 					(unit 1)
 				)
@@
 			)
 		)
-		(property "Value" "100n"
+		(property "Value" "10u"
 			(at 214.63 63.5 90)
 			(show_name no)
@@
 		(dnp no)
 		(fields_autoplaced yes)
-		(property "Reference" "R6"
+		(property "Reference" "R2"
 			(at 101.6 144.78 90)
 			(show_name no)
@@
 			(project "Double-DigiPot-with-IR"
 				(path "/8790fbe4-afd7-47db-a1db-a7a2fdad799c"
-					(reference "R6")
+					(reference "R2")
 					(unit 1)
 				)
